Commit message: update: rviz file and fix control error

File: xmen_description/urdf/cctv.urdf (robot description, URDF)
Before this commit: robot assembly_1, 30 links, 29 joints
Joints:
- joint camera_mount_joint: origin xyz=0 -0.0045 0 rpy=0 0 -1.5707963267948966 -> xyz=0 0.0205 0 rpy=0 0 1.5707963267948966
